Commit message: Items Adjusted
All items now have max mass of 1.5. Friction on cup decreased and bowl size reduced.

File: items/00.urdf (robot description, URDF)
Before this commit: robot urdf_robot, 1 links, 0 joints
Links:
- link base_link: mass 10 -> 1.0; geometry collision mesh filename=bowl.obj scale=0.3 0.3 0.3; visual mesh filename=bowl.obj scale=0.3 0.3 0.3

File: items/01.urdf (robot description, URDF)
Before this commit: robot cube.urdf, 1 links, 0 joints
Links:
- link baseLink: mass 15 -> 1.5

File: items/04.urdf (robot description, URDF)
Before this commit: robot urdf_robot, 1 links, 0 joints
Links:
- link base_link: mass 5 -> 1

File: items/05.urdf (robot description, URDF)
Before this commit: robot cube.urdf, 1 links, 0 joints
Links:
- link baseLink: mass 10 -> 1

File: items/06.urdf (robot description, URDF)
Before this commit: robot urdf_robot, 1 links, 0 joints
Links:
- link base_link: mass 5 -> 1
